Commit message: ibvs push 1

File: src/picar_description/urdf/picar_tracking.urdf (robot description, URDF)
Before this commit: robot picar_tracking, 7 links, 6 joints
Links:
- added link car_base
- added link pan_link; visual cylinder length=0.05 radius=0.008
- added link tilt_link; visual cylinder length=0.03 radius=0.008
Joints:
- removed joint mount_to_chassis
- added joint camera_optical_joint: type fixed, parent tilt_link, child camera, origin xyz=0.0 -0.015 0.0 rpy=0 0 0
- added joint car_base_to_chassis: type fixed, parent car_base, child base_link, origin xyz=0.0 0.0 -0.05 rpy=0 0 0
- added joint pan_joint: type revolute, parent car_base, child pan_link, origin xyz=0.0 -0.060 0.0 rpy=0 0 0, axis 0 1 0, limit lower=-1.5708 upper=1.5708 effort=1.0 velocity=1.0
- added joint tilt_joint: type revolute, parent pan_link, child tilt_link, origin xyz=0.0 -0.020 0.0 rpy=0 0 0, axis 1 0 0, limit lower=-0.6109 upper=0.6109 effort=1.0 velocity=1.0
